File: display-adapter-v2.kicad_sch (KiCad schematic)
At the start: 9 parts, among them J1 Display_In, J2 Inky_Left_1_20, J3 Inky_Right_21_40, J4 Display_Out_2, J5 Display_Out_3, J6 Display_Out_4

Commit message: bugfix: wrong 1x21 instead of 1x20 footprint for Inky-connectors
Parts:
- J2, J3: footprint Connector_PinHeader_2.54mm:PinHeader_1x21_P2.54mm_Vertical -> Connector_PinHeader_2.54mm:PinHeader_1x20_P2.54mm_Vertical
Changed lines of the file:
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@@
   (title_block
     (title "Display-Adapter-v2")
-    (date "2026-02-23")
-    (rev "1.00")
+    (date "2026-03-10")
+    (rev "1.01")
     (company "Bernhard Bablok")
     (comment 1 "https://github.com/bablokb/pcb-datalogger-display-adapter-v2")
@@
       (effects (font (size 1.27 1.27)) (justify left))
     )
-    (property "Footprint" "Connector_PinHeader_2.54mm:PinHeader_1x21_P2.54mm_Vertical" (at 86.995 60.325 0)
+    (property "Footprint" "Connector_PinHeader_2.54mm:PinHeader_1x20_P2.54mm_Vertical" (at 86.995 60.325 0)
       (effects (font (size 1.27 1.27)) hide)
     )
@@
       (effects (font (size 1.27 1.27)) (justify left))
     )
-    (property "Footprint" "Connector_PinHeader_2.54mm:PinHeader_1x21_P2.54mm_Vertical" (at 112.395 62.865 0)
-      (effects (font (size 1.27 1.27)) hide)
-    )
+    (property "Footprint" "Connector_PinHeader_2.54mm:PinHeader_1x20_P2.54mm_Vertical" (at 112.395 62.865 0)
+      (effects (font (size 1.27 1.27)) hide)
+    )
